Commit message: 20230907AddLivoxLidars

File: livox_sim/urdf/livox_avia.xacro (robot description, xacro)
@@ -85,5 +85,5 @@
     </gazebo>
   </xacro:macro>
-  <xacro:macro name="Livox_AVIA" params="visualize:=True name:=livox">
+  <xacro:macro name="Livox_AVIA" params="*origin visualize:=True name:=livox">
   <joint name="${name}_base_mount_joint" type="fixed">
       <xacro:insert_block name="origin" />

File: livox_sim/urdf/livox_mid360.xacro (robot description, xacro)
@@ -58,5 +58,5 @@
     </gazebo>
   </xacro:macro>
-  <xacro:macro name="Livox_Mid40" params="visualize:=True name:=livox">
+  <xacro:macro name="Livox_Mid40" params="*origin visualize:=True name:=livox">
   <joint name="${name}_base_mount_joint" type="fixed">
       <xacro:insert_block name="origin" />

File: smb_simulator/smb_description/urdf/sensor_head.urdf.xacro (robot description, xacro)
@@ -29,7 +29,9 @@
 		<!-- <xacro:include filename="$(find livox_laser_simulation)/urdf/livox_avia.xacro"/>
 		<xacro:Livox_AVIA name="livox_avia">
+		<origin xyz="0.1 0.1 0.5" rpy="0 0 0" />
 		</xacro:Livox_AVIA> -->
 		<xacro:include filename="$(find livox_laser_simulation)/urdf/livox_mid360.xacro"/>
 		<xacro:Livox_Mid40 name="livox_mid360">
+		<origin xyz="0.2 0.00 0.5" rpy="0 0.5 0" />
 		</xacro:Livox_Mid40>
 		<xacro:include filename="$(find smb_description)/urdf/smb_rgb_camera.urdf.xacro"/>
