Commit message: 20230907AddLivoxLidars

File: livox_sim/urdf/livox_mid360.xacro (robot description, xacro)
@@ -2,5 +2,5 @@
 <robot xmlns:xacro="http://ros.org/wiki/xacro">
   <xacro:property name="M_PI" value="3.14159"/>
-  <xacro:property name="laser_min_range" value="0.1"/>
+  <xacro:property name="laser_min_range" value="0.7"/>
   <xacro:property name="laser_max_range" value="200.0"/>
   <xacro:property name="ros_topic" value="scan"/>

File: smb_simulator/smb_description/urdf/sensor_head.urdf.xacro (robot description, xacro)
@@ -27,12 +27,12 @@
 			<origin xyz="0.1 0.3 -0.1" rpy="0 0.5 0" />
 		</xacro:BPearl> -->
-		<!-- <xacro:include filename="$(find livox_laser_simulation)/urdf/livox_avia.xacro"/>
+		<xacro:include filename="$(find livox_laser_simulation)/urdf/livox_avia.xacro"/>
 		<xacro:Livox_AVIA name="livox_avia">
-		<origin xyz="0.1 0.1 0.5" rpy="0 0 0" />
-		</xacro:Livox_AVIA> -->
-		<xacro:include filename="$(find livox_laser_simulation)/urdf/livox_mid360.xacro"/>
+		<origin xyz="0.2 0.0 0.5" rpy="0 0 0" />
+		</xacro:Livox_AVIA>
+		<!-- <xacro:include filename="$(find livox_laser_simulation)/urdf/livox_mid360.xacro"/>
 		<xacro:Livox_Mid40 name="livox_mid360">
 		<origin xyz="0.2 0.00 0.5" rpy="0 0.5 0" />
-		</xacro:Livox_Mid40>
+		</xacro:Livox_Mid40> -->
 		<xacro:include filename="$(find smb_description)/urdf/smb_rgb_camera.urdf.xacro"/>
 		<!-- Cameras: -->
