Commit message: 20230907AddLivoxLidars

File: smb_simulator/smb_description/urdf/sensor_head.urdf.xacro (robot description, xacro)
@@ -23,4 +23,14 @@
 			<origin xyz="0.1 -0.3 -0.1" rpy="0 0.5 0" />
 		</xacro:OS1-64>
+		<!-- <xacro:include filename="$(find lidar_description)/urdf/BPearl.urdf.xacro"/>
+		<xacro:BPearl parent="${name}_base_link" name="BPearl" topic="BPearl_points" hz="10" lasers="16" samples="1875" min_range="0.7">
+			<origin xyz="0.1 0.3 -0.1" rpy="0 0.5 0" />
+		</xacro:BPearl> -->
+		<!-- <xacro:include filename="$(find livox_laser_simulation)/urdf/livox_avia.xacro"/>
+		<xacro:Livox_AVIA name="livox_avia">
+		</xacro:Livox_AVIA> -->
+		<xacro:include filename="$(find livox_laser_simulation)/urdf/livox_mid360.xacro"/>
+		<xacro:Livox_Mid40 name="livox_mid360">
+		</xacro:Livox_Mid40>
 		<xacro:include filename="$(find smb_description)/urdf/smb_rgb_camera.urdf.xacro"/>
 		<!-- Cameras: -->

Commit message: 20230909

File: smb_simulator/smb_description/urdf/sensor_head.urdf.xacro (robot description, xacro)
@@ -27,12 +27,16 @@
 			<origin xyz="0.1 0.3 -0.1" rpy="0 0.5 0" />
 		</xacro:BPearl> -->
-		<xacro:include filename="$(find livox_laser_simulation)/urdf/livox_avia.xacro"/>
+		<!-- <xacro:include filename="$(find livox_laser_simulation)/urdf/livox_avia.xacro"/>
 		<xacro:Livox_AVIA name="livox_avia">
-		<origin xyz="0.2 0.0 0.5" rpy="0 0 0" />
-		</xacro:Livox_AVIA>
+		<origin xyz="0.2 0.0 0.5" rpy="0 0.5 0" />
+		</xacro:Livox_AVIA> -->
 		<!-- <xacro:include filename="$(find livox_laser_simulation)/urdf/livox_mid360.xacro"/>
 		<xacro:Livox_Mid40 name="livox_mid360">
 		<origin xyz="0.2 0.00 0.5" rpy="0 0.5 0" />
 		</xacro:Livox_Mid40> -->
+		<xacro:include filename="$(find lidar_description)/urdf/HDL-32E.urdf.xacro"/>
+		<xacro:HDL-32E parent="${name}_base_link" name="lidar_back" topic="lidar_back_points" hz="10" lasers="32" samples="440" min_range="1.0">
+			<origin xyz="-0.05 0.3 -0.1" rpy="0 -0.5 0" />
+		</xacro:HDL-32E>
 		<xacro:include filename="$(find smb_description)/urdf/smb_rgb_camera.urdf.xacro"/>
 		<!-- Cameras: -->

Commit message: 20231017

File: smb_simulator/smb_description/urdf/sensor_head.urdf.xacro (robot description, xacro)
@@ -39,4 +39,8 @@
 			<origin xyz="-0.05 0.3 -0.1" rpy="0 -0.5 0" />
 		</xacro:HDL-32E>
+		<!-- <xacro:include filename="$(find lidar_description)/urdf/BPearl.urdf.xacro"/>
+		<xacro:BPearl parent="${name}_base_link" name="lidar_back" topic="lidar_back_points" hz="10" lasers="64" samples="440" min_range="1.0">
+			<origin xyz="-0.1 0.3 -0.1" rpy="0 -0.9 0" />
+		</xacro:BPearl> -->
 		<xacro:include filename="$(find smb_description)/urdf/smb_rgb_camera.urdf.xacro"/>
 		<!-- Cameras: -->
