Commit message: ImproveTheSmbAndRelativeUrdfFiles. 20241105

File: smb_simulator/smb_description/urdf/sensor_head_2.urdf.xacro (robot description, xacro)
@@ -16,11 +16,17 @@
 		<xacro:arg name="gpu" default="true"/>
 		<xacro:include filename="$(find lidar_description)/urdf/VLP-16-2.urdf.xacro"/>
-		<xacro:VLP-16 parent="${name}_base_link" name="${name}_velodyne" topic="${name}_velodyne_points" hz="10" lasers="32" samples="440" gpu="$(arg gpu)" collision_range="0.2" min_range="0.2" RobotNs="${RobotNs}">
+		<xacro:VLP-16 parent="${name}_base_link" name="${name}_Top_velodyne" topic="${name}_Top_velodyne_points" hz="10" lasers="32" samples="440" gpu="$(arg gpu)" collision_range="0.2" min_range="0.2" RobotNs="${RobotNs}">
 			<origin xyz="0.03 0 0.08" rpy="0 0 0" />
 		</xacro:VLP-16>
-		<xacro:include filename="$(find lidar_description)/urdf/OS1-64-3.urdf.xacro"/>
+		<xacro:VLP-16 parent="${name}_base_link" name="${name}_Front_velodyne" topic="${name}_Front_velodyne_points" hz="10" lasers="32" samples="440" gpu="false" collision_range="0.2" min_range="0.7" RobotNs="${RobotNs}">
+			<origin xyz="0.1 -0.3 -0.1" rpy="0 0.5 0" />
+		</xacro:VLP-16>
+		<xacro:VLP-16 parent="${name}_base_link" name="${name}_Back_velodyne" topic="${name}_Back_velodyne_points" hz="10" lasers="32" samples="440" gpu="false" collision_range="0.2" min_range="1.0" RobotNs="${RobotNs}">
+			<origin xyz="-0.05 0.3 -0.1" rpy="0 -0.5 0" />
+		</xacro:VLP-16>
+		<!-- <xacro:include filename="$(find lidar_description)/urdf/OS1-64-3.urdf.xacro"/>
 		<xacro:OS1-64-3 parent="${name}_base_link" name="${name}_lidar_front" topic="${name}_lidar_front_points" hz="10" lasers="32" samples="440" min_range="0.7">
 			<origin xyz="0.1 -0.3 -0.1" rpy="0 0.5 0" />
-		</xacro:OS1-64-3>
+		</xacro:OS1-64-3> -->
 		<!-- <xacro:include filename="$(find smb_description)/urdf/depthCamera.xacro"/>
 		<xacro:depthCamera parent="${name}_base_link" camID="1" name="face">
@@ -43,8 +49,8 @@
 		<origin xyz="0.2 0.00 0.5" rpy="0 0.5 0" />
 		</xacro:Livox_Mid40> -->
-		<xacro:include filename="$(find lidar_description)/urdf/HDL-32E.urdf.xacro"/>
+		<!-- <xacro:include filename="$(find lidar_description)/urdf/HDL-32E.urdf.xacro"/>
 		<xacro:HDL-32E parent="${name}_base_link" name="${name}_lidar_back" topic="${name}_lidar_back_points" hz="10" lasers="32" samples="440" min_range="1.0">
 			<origin xyz="-0.05 0.3 -0.1" rpy="0 -0.5 0" />
-		</xacro:HDL-32E>
+		</xacro:HDL-32E> -->
 		<!-- <xacro:include filename="$(find lidar_description)/urdf/BPearl.urdf.xacro"/>
 		<xacro:BPearl parent="${name}_base_link" name="lidar_back" topic="lidar_back_points" hz="10" lasers="64" samples="440" min_range="1.0">

File: smb_simulator/smb_description/urdf/smb.urdf.xacro (robot description, xacro)
@@ -82,6 +82,6 @@
 		</plugin>
 	</gazebo>
-	<xacro:include filename="$(find smb_description)/urdf/sensor_head_2.urdf.xacro"/>
-	<xacro:sensor_head parent="$(arg robot_namespace)_base_link" name="$(arg robot_namespace)_sensor_head" RobotNs="$(arg robot_namespace)">
+	<xacro:include filename="$(find smb_description)/urdf/SensorHead.urdf.xacro"/>
+	<xacro:sensor_head parent="$(arg robot_namespace)_base_link" name="$(arg robot_namespace)_Sensor_Head" RobotNs="$(arg robot_namespace)">
 		<origin xyz="0.2 0 0.576" rpy="0 0 0" />
 	</xacro:sensor_head>
