Commit message: Try to equip Smb with depth cameras, but fail. 20241106.

File: smb_simulator/smb_description/urdf/SensorHead.urdf.xacro (robot description, xacro)
@@ -25,4 +25,11 @@
 			<origin xyz="-0.05 0.3 -0.1" rpy="0 -0.5 0" />
 		</xacro:VLP-16> -->
+		<!-- <xacro:include filename="$(find smb_description)/urdf/depthCamera.xacro"/>
+		<xacro:depthCamera parent="${name}_base_link" name="${name}_Front">
+        	<origin rpy="0 0 0" xyz="0.9 -0.0125 0.15"/>
+    	</xacro:depthCamera>
+		<xacro:depthCamera parent="${name}_base_link" name="${name}_Back">
+        	<origin rpy="0 0 0" xyz="-0.9 -0.0125 0.15"/>
+    	</xacro:depthCamera> -->
 	</xacro:macro>
 </robot>

File: smb_simulator/smb_description/urdf/depthCamera.xacro (robot description, xacro)
@@ -1,11 +1,11 @@
 <?xml version="1.0"?>
 <robot xmlns:xacro="http://www.ros.org/wiki/xacro">
-    <xacro:macro name="depthCamera" params="parent camID name *origin">
-        <joint name="camera_joint_${name}" type="fixed">
+    <xacro:macro name="depthCamera" params="parent name *origin">
+        <joint name="${name}_DepthCamera_joint" type="fixed">
             <xacro:insert_block name="origin"/>
             <parent link="${parent}"/>
-            <child link="camera_${name}"/>
+            <child link="${name}_DepthCamera"/>
         </joint>
-        <link name="camera_${name}">
+        <link name="${name}_DepthCamera">
             <collision>
             <origin xyz="0 0 0" rpy="0 0 0"/>
@@ -26,14 +26,14 @@
             </inertial>
         </link>
-        <joint name="camera_optical_joint_${name}" type="fixed">
+        <joint name="${name}_DepthCamera_optical_joint" type="fixed">
             <origin xyz="0 0 0" rpy="${-pi/2} 0 ${-pi/2}"/>
-            <parent link="camera_${name}"/>
-            <child link="camera_optical_${name}"/>
+            <parent link="${name}_DepthCamera"/>
+            <child link="${name}_DepthCamera_optical"/>
         </joint>
-        <link name="camera_optical_${name}">
+        <link name="${name}_DepthCamera_optical">
         </link>
-        <gazebo reference="camera_${name}">
+        <gazebo reference="${name}_DepthCamera">
             <!-- <material>Gazebo/Black</material> -->
-            <sensor name="camera_${name}_camera" type="depth">
+            <sensor name="${name}_DepthCamera_sensor" type="depth">
                 <update_rate>16</update_rate>
                 <camera>
@@ -49,16 +49,16 @@
                     </clip>
                 </camera>
-                <plugin name="camera_${name}_controller" filename="libgazebo_ros_openni_kinect.so">
+                <plugin name="camera_controller" filename="libgazebo_ros_openni_kinect.so">
                     <baseline>0.025</baseline>
                     <alwaysOn>true</alwaysOn>
-                    <updateRate>0.0</updateRate>
-                    <cameraName>camera_${name}</cameraName>
-                    <imageTopicName>/camera_${name}/color/image_raw</imageTopicName>
-                    <cameraInfoTopicName>/camera_${name}/color/camera_info</cameraInfoTopicName>
-                    <depthImageTopicName>/camera_${name}/depth/image_raw</depthImageTopicName>
-                    <depthImageInfoTopicName>/camera_${name}/depth/camera_info</depthImageInfoTopicName>
+                    <updateRate>1.0</updateRate>
+                    <cameraName>${name}_DepthCamera</cameraName>
+                    <imageTopicName>${name}_DepthCamera/color/image_raw</imageTopicName>
+                    <cameraInfoTopicName>${name}_DepthCamera/color/camera_info</cameraInfoTopicName>
+                    <depthImageTopicName>${name}_DepthCamera/depth/image_raw</depthImageTopicName>
+                    <depthImageInfoTopicName>${name}_DepthCamera/depth/camera_info</depthImageInfoTopicName>
                     <!-- <pointCloudTopicName>/camera_${name}/depth/points</pointCloudTopicName> -->
-                    <pointCloudTopicName>/cam${camID}/point_cloud_${name}</pointCloudTopicName>
-                    <frameName>camera_optical_${name}</frameName>
+                    <pointCloudTopicName>${name}_DepthCamera/depth/points</pointCloudTopicName>
+                    <frameName>${name}_DepthCamera_optical</frameName>
                     <pointCloudCutoff>0.3</pointCloudCutoff>
                     <pointCloudCutoffMax>3.9</pointCloudCutoffMax>

Commit message: Add realsense gazebo into the simulator. 20241106

File: smb_simulator/smb_description/urdf/SensorHead.urdf.xacro (robot description, xacro)
@@ -27,9 +27,13 @@
 		<!-- <xacro:include filename="$(find smb_description)/urdf/depthCamera.xacro"/>
 		<xacro:depthCamera parent="${name}_base_link" name="${name}_Front">
-        	<origin rpy="0 0 0" xyz="0.9 -0.0125 0.15"/>
-    	</xacro:depthCamera>
-		<xacro:depthCamera parent="${name}_base_link" name="${name}_Back">
+        	<origin rpy="0 0.7 0" xyz="0.9 -0.0125 0.15"/>
+    	</xacro:depthCamera> -->
+		<!-- <xacro:depthCamera parent="${name}_base_link" name="${name}_Back">
         	<origin rpy="0 0 0" xyz="-0.9 -0.0125 0.15"/>
     	</xacro:depthCamera> -->
+		<xacro:include filename="$(find realsense_simulator)/xacro/depthcam.xacro"/>
+		<xacro:realsense_d435 sensor_name="${name}_Front_RealsenseD435" parent_link="${name}_base_link" rate="10">
+    		<origin rpy="0 0.3 0 " xyz="0.15 0 -0.15"/>
+  		</xacro:realsense_d435>
 	</xacro:macro>
 </robot>

File: unitree_simulator/unitree_ros/robots/a1_description/xacro/SensorHeadForUnitreeA1.urdf.xacro (robot description, xacro)
@@ -32,4 +32,8 @@
         	<origin rpy="0 0 0" xyz="-0.9 -0.0125 0.15"/>
     	</xacro:depthCamera> -->
+		<xacro:include filename="$(find realsense_simulator)/xacro/depthcam.xacro"/>
+		<xacro:realsense_d435 sensor_name="${name}_Front_RealsenseD435" parent_link="${name}_base_link" rate="10">
+    		<origin rpy="0 0.16 0 " xyz="0.25 0 -0.05"/>
+  		</xacro:realsense_d435>
 	</xacro:macro>
 </robot>
