Commit message: 20240505

File: unitree_simulator/unitree_ros/robots/a1_description/xacro/depthCamera.xacro (robot description, xacro)
@@ -62,5 +62,5 @@
                     <frameName>camera_optical_${name}</frameName>
                     <pointCloudCutoff>0.3</pointCloudCutoff>
-                    <pointCloudCutoffMax>3.5</pointCloudCutoffMax>
+                    <pointCloudCutoffMax>3.9</pointCloudCutoffMax>
                     <distortionK1>0.0</distortionK1>
                     <distortionK2>0.0</distortionK2>

File: unitree_simulator/unitree_ros/robots/a1_description/xacro/robot.xacro (robot description, xacro)
@@ -141,5 +141,5 @@
 	</xacro:sensor_head> -->
     <xacro:depthCamera camID="1" name="face">
-        <origin rpy="${PI} 0 0" xyz="0.35 0.0125 0.15"/>
+        <origin rpy="${PI} 0 0" xyz="0.25 0.0125 0.15"/>
     </xacro:depthCamera>
     <xacro:depthCamera camID="2" name="chin">
@@ -153,5 +153,5 @@
     </xacro:depthCamera>
     <xacro:depthCamera camID="5" name="rearDown">
-        <origin rpy="${PI} 0.2618 ${PI}" xyz="-0.35 -0.0125 0.15"/>
+        <origin rpy="${PI} 0.2618 ${PI}" xyz="-0.25 -0.0125 0.15"/>
     </xacro:depthCamera>
 </robot>
