Commit message: 20240306

File: unitree_simulator/unitree_ros/robots/a1_description/xacro/robot.xacro (robot description, xacro)
@@ -17,8 +17,8 @@
             <origin rpy="0 0 0" xyz="0 0 0"/>
             <parent link="world"/>
-            <child link="base"/>
+            <child link="base_link"/>
         </joint>
     </xacro:if>
-    <link name="base">
+    <link name="base_link">
         <visual>
             <origin rpy="0 0 0" xyz="0 0 0"/>
@@ -30,5 +30,5 @@
     <joint name="floating_base" type="fixed">
         <origin rpy="0 0 0" xyz="0 0 0"/>
-        <parent link="base"/>
+        <parent link="base_link"/>
         <child link="trunk"/>
     </joint>
@@ -127,5 +127,5 @@
         <alwaysOn>true</alwaysOn>
         <updateRate>50.0</updateRate>
-        <bodyName>base</bodyName>
+        <bodyName>base_link</bodyName>
         <topicName>ground_truth/state</topicName>
         <gaussianNoise>0.01</gaussianNoise>

Commit message: 20240306

File: unitree_simulator/unitree_ros/robots/a1_description/xacro/robot.xacro (robot description, xacro)
@@ -125,13 +125,17 @@
     <gazebo>
         <plugin name="p3d_base_controller" filename="libgazebo_ros_p3d.so">
-        <alwaysOn>true</alwaysOn>
-        <updateRate>50.0</updateRate>
-        <bodyName>base_link</bodyName>
-        <topicName>ground_truth/state</topicName>
-        <gaussianNoise>0.01</gaussianNoise>
-        <frameName>world</frameName>
-        <xyzOffsets>0 0 0</xyzOffsets>
-        <rpyOffsets>0 0 0</rpyOffsets>
-    </plugin>
-</gazebo>
+            <alwaysOn>true</alwaysOn>
+            <updateRate>50.0</updateRate>
+            <bodyName>base_link</bodyName>
+            <topicName>ground_truth/state</topicName>
+            <gaussianNoise>0.01</gaussianNoise>
+            <frameName>world</frameName>
+            <xyzOffsets>0 0 0</xyzOffsets>
+            <rpyOffsets>0 0 0</rpyOffsets>
+        </plugin>
+    </gazebo>
+    <xacro:include filename="$(find a1_description)/xacro/sensor_head.urdf.xacro"/>
+	<xacro:sensor_head parent="base_link" name="sensor_head">
+		<origin xyz="0.0 0 0.0" rpy="0 0 0" />
+	</xacro:sensor_head>
 </robot>

Commit message: 20240313

File: unitree_simulator/unitree_ros/robots/a1_description/xacro/robot.xacro (robot description, xacro)
@@ -7,4 +7,5 @@
     <xacro:include filename="$(find a1_description)/xacro/stairs.xacro"/>
     <xacro:include filename="$(find a1_description)/xacro/gazebo.xacro"/>
+    <xacro:include filename="$(find a1_description)/xacro/depthCamera.xacro"/>
     <!-- <xacro:include filename="$(find a1_gazebo)/launch/stairs.urdf.xacro"/> -->
     <!-- <xacro:stairs stairs="15" xpos="0" ypos="0" zpos="0" /> -->
@@ -135,7 +136,22 @@
         </plugin>
     </gazebo>
-    <xacro:include filename="$(find a1_description)/xacro/sensor_head.urdf.xacro"/>
+    <!-- <xacro:include filename="$(find a1_description)/xacro/sensor_head.urdf.xacro"/>
 	<xacro:sensor_head parent="base_link" name="sensor_head">
 		<origin xyz="0.0 0 0.0" rpy="0 0 0" />
-	</xacro:sensor_head>
+	</xacro:sensor_head> -->
+    <xacro:depthCamera camID="1" name="face">
+        <origin rpy="${PI} 0 0" xyz="0.35 0.0125 0.15"/>
+    </xacro:depthCamera>
+    <xacro:depthCamera camID="2" name="chin">
+        <origin rpy="${PI} ${PI/2} 0" xyz="0.2522 0.0125 0.0"/>
+    </xacro:depthCamera>
+    <xacro:depthCamera camID="3" name="left">
+        <origin rpy="${PI} 0.2618 ${PI/2}" xyz="0.0 0.15 -0.0176"/>
+    </xacro:depthCamera>
+    <xacro:depthCamera camID="4" name="right">
+        <origin rpy="${PI} 0.2618 ${-PI/2}" xyz="0.0 -0.15 -0.0176"/>
+    </xacro:depthCamera>
+    <xacro:depthCamera camID="5" name="rearDown">
+        <origin rpy="${PI} 0.2618 ${PI}" xyz="-0.35 -0.0125 0.15"/>
+    </xacro:depthCamera>
 </robot>

Commit message: 20240505

File: unitree_simulator/unitree_ros/robots/a1_description/xacro/robot.xacro (robot description, xacro)
@@ -141,5 +141,5 @@
 	</xacro:sensor_head> -->
     <xacro:depthCamera camID="1" name="face">
-        <origin rpy="${PI} 0 0" xyz="0.25 0.0125 0.15"/>
+        <origin rpy="${PI} 0 0" xyz="0.2 0.0125 0.15"/>
     </xacro:depthCamera>
     <xacro:depthCamera camID="2" name="chin">
@@ -153,5 +153,5 @@
     </xacro:depthCamera>
     <xacro:depthCamera camID="5" name="rearDown">
-        <origin rpy="${PI} 0.2618 ${PI}" xyz="-0.25 -0.0125 0.15"/>
+        <origin rpy="${PI} 0.2618 ${PI}" xyz="-0.2 -0.0125 0.15"/>
     </xacro:depthCamera>
 </robot>
