Commit message: Equip Unitree A1 Robot with just one Velodyne lidar. 20241106.

File: unitree_simulator/unitree_ros/robots/a1_description/xacro/RobotForPPCupy.xacro (robot description, xacro)
@@ -5,11 +5,6 @@
     <xacro:include filename="$(find a1_description)/xacro/materials.xacro"/>
     <xacro:include filename="$(find a1_description)/xacro/leg.xacro"/>
-    <xacro:include filename="$(find a1_description)/xacro/stairs.xacro"/>
     <xacro:include filename="$(find a1_description)/xacro/gazebo.xacro"/>
-    <xacro:include filename="$(find a1_description)/xacro/depthCamera.xacro"/>
-    <!-- <xacro:include filename="$(find a1_gazebo)/launch/stairs.urdf.xacro"/> -->
-    <!-- <xacro:stairs stairs="15" xpos="0" ypos="0" zpos="0" /> -->
-    <!-- Rollover Protection mode will add an additional stick on the top, use "true" or "false" to switch it. -->
-    <xacro:property name="rolloverProtection" value="false"/>
+    <!-- <xacro:include filename="$(find a1_description)/xacro/depthCamera.xacro"/> -->
     <!-- Debug mode will hung up the robot, use "true" or "false" to switch it. -->
     <xacro:if value="$(arg DEBUG)">
@@ -57,33 +52,4 @@
         </inertial>
     </link>
-    <xacro:if value="${(rolloverProtection == 'true')}">
-        <joint name="stick_joint" type="fixed">
-            <parent link="trunk"/>
-            <child link="stick_link"/>
-            <origin rpy="0 0 0" xyz="${0.18} 0 ${stick_length/2.0+0.08}"/>
-        </joint>
-        <link name="stick_link">
-            <visual>
-                <geometry>
-                    <cylinder length="${stick_length}" radius="${stick_radius}"/>
-                </geometry>
-                <origin rpy="0 0 0" xyz="0 0 0"/>
-                <material name="white"/>
-            </visual>
-            <collision>
-                <geometry>
-                    <cylinder length="${stick_length}" radius="${stick_radius}"/>
-                </geometry>
-                <origin rpy="0 0 0" xyz="0 0 0"/>
-            </collision>
-            <inertial>
-                <mass value="${stick_mass}"/>
-                <inertia
-                    ixx="${stick_mass / 2.0 * (stick_radius*stick_radius)}" ixy="0.0" ixz="0.0"
-                    iyy="${stick_mass / 12.0 * (3*stick_radius*stick_radius + stick_length*stick_length)}" iyz="0.0"
-                    izz="${stick_mass / 12.0 * (3*stick_radius*stick_radius + stick_length*stick_length)}"/>
-            </inertial>
-        </link>
-    </xacro:if>
     <joint name="imu_joint" type="fixed">
         <parent link="trunk"/>
@@ -123,5 +89,4 @@
         <origin rpy="0 0 0" xyz="${-leg_offset_x} ${leg_offset_y} 0"/>
     </xacro:leg>
-    <!-- <xacro:stairs stairs="15" xpos="0" ypos="2.0" zpos="0" /> -->
     <gazebo>
         <plugin name="p3d_base_controller" filename="libgazebo_ros_p3d.so">
@@ -140,5 +105,9 @@
 		<origin xyz="0.0 0 0.0" rpy="0 0 0" />
 	</xacro:sensor_head> -->
-    <xacro:depthCamera camID="1" name="face">
+    <xacro:include filename="$(find a1_description)/xacro/SensorHeadForUnitreeA1.urdf.xacro"/>
+	<xacro:sensor_head parent="base_link" name="Sensor_Head">
+		<origin xyz="0.0 0 0.03" rpy="0 0 0" />
+	</xacro:sensor_head>
+    <!-- <xacro:depthCamera camID="1" name="face">
         <origin rpy="${PI} 0 0" xyz="0.2 0.0125 0.15"/>
     </xacro:depthCamera>
@@ -154,4 +123,4 @@
     <xacro:depthCamera camID="5" name="rearDown">
         <origin rpy="${PI} 0.2618 ${PI}" xyz="-0.2 -0.0125 0.15"/>
-    </xacro:depthCamera>
+    </xacro:depthCamera> -->
 </robot>
