Commit message: Try to spawn two smb robots but failed as the controllers has not been equipped well in 20241103.

File: lidar_simulator/lidar_description/urdf/OS1-64-3.urdf.xacro (robot description, xacro)
@@ -3,5 +3,5 @@
   <xacro:property name="M_PI" value="3.1415926535897931" />
   <xacro:macro name="OS1-64-3" params="*origin parent:=base_link name:=os1_sensor topic:=/os1_cloud_node/points hz:=10 lasers:=64 samples:=512 collision_range:=0.7 min_range:=0.225 max_range:=100.0 noise:=0.008 min_angle:=-${M_PI} max_angle:=${M_PI} gpu:=false">
-    <joint name="mount_joint" type="fixed">
+    <joint name="${name}_mount_joint" type="fixed">
       <xacro:insert_block name="origin" />
       <parent link="${parent}"/>
@@ -28,16 +28,16 @@
       </visual>
     </link>
-    <link name="os1_3_imu" />
-    <link name="os1_3_lidar" />
-    <joint name="imu_link_joint" type="fixed">
+    <link name="${name}_os1_3_imu" />
+    <link name="${name}_os1_3_lidar" />
+    <joint name="${name}_imu_link_joint" type="fixed">
       <parent link="${name}" />
-      <child link="os1_3_imu" />
+      <child link="${name}_os1_3_imu" />
       <origin xyz="0.006253 -0.011775 0.007645" rpy="0 0 0" />
     </joint>
-    <gazebo reference="os1_3_imu">
+    <gazebo reference="${name}_os1_3_imu">
     </gazebo>
-    <joint name="lidar_link_joint" type="fixed">
+    <joint name="${name}_lidar_link_joint" type="fixed">
       <parent link="${name}" />
-      <child link="os1_3_lidar" />
+      <child link="${name}_os1_3_lidar" />
       <origin xyz="0.0 0.0 0.03618" rpy="0 0 0" />
     </joint>
@@ -118,5 +118,5 @@
     <gazebo>
       <plugin name="imu_controller" filename="libhector_gazebo_ros_imu.so">
-        <robotNamespace>/</robotNamespace>
+        <robotNamespace>/${name}</robotNamespace>
         <updateRate>100.0</updateRate>
         <bodyName>os1_3_imu</bodyName>

File: smb_simulator/smb_description/urdf/sensor_head_2.urdf.xacro (robot description, xacro)
@@ -16,9 +16,9 @@
 		<xacro:arg name="gpu" default="true"/>
 		<xacro:include filename="$(find lidar_description)/urdf/VLP-16-2.urdf.xacro"/>
-		<xacro:VLP-16 parent="${name}_base_link" name="velodyne" topic="velodyne_points" hz="10" lasers="32" samples="440" gpu="$(arg gpu)" collision_range="0.2" min_range="0.2">
+		<xacro:VLP-16 parent="${name}_base_link" name="${name}_velodyne" topic="${name}_velodyne_points" hz="10" lasers="32" samples="440" gpu="$(arg gpu)" collision_range="0.2" min_range="0.2">
 			<origin xyz="0.03 0 0.08" rpy="0 0 0" />
 		</xacro:VLP-16>
 		<xacro:include filename="$(find lidar_description)/urdf/OS1-64-3.urdf.xacro"/>
-		<xacro:OS1-64-3 parent="${name}_base_link" name="lidar_front" topic="lidar_front_points" hz="10" lasers="32" samples="440" min_range="0.7">
+		<xacro:OS1-64-3 parent="${name}_base_link" name="${name}_lidar_front" topic="${name}_lidar_front_points" hz="10" lasers="32" samples="440" min_range="0.7">
 			<origin xyz="0.1 -0.3 -0.1" rpy="0 0.5 0" />
 		</xacro:OS1-64-3>
@@ -44,5 +44,5 @@
 		</xacro:Livox_Mid40> -->
 		<xacro:include filename="$(find lidar_description)/urdf/HDL-32E.urdf.xacro"/>
-		<xacro:HDL-32E parent="${name}_base_link" name="lidar_back" topic="lidar_back_points" hz="10" lasers="32" samples="440" min_range="1.0">
+		<xacro:HDL-32E parent="${name}_base_link" name="${name}_lidar_back" topic="${name}_lidar_back_points" hz="10" lasers="32" samples="440" min_range="1.0">
 			<origin xyz="-0.05 0.3 -0.1" rpy="0 -0.5 0" />
 		</xacro:HDL-32E>

File: smb_simulator/smb_description/urdf/smb_old.urdf.xacro (robot description, xacro)
@@ -13,5 +13,5 @@
 	<xacro:include filename="$(find smb_description)/urdf/smb_utils.urdf.xacro" />
 	<!-- Base link is the robot chassis -->
-	<link name="$(arg robot_namespace)_base_link">
+	<link name="base_link">
 		<!-- <visual>
 			<origin xyz="0 0 0" rpy="0 0 0" />
@@ -37,9 +37,9 @@
 		</collision>
 	</link>
-	<gazebo reference="$(arg robot_namespace)_base_link">
+	<gazebo reference="base_link">
 		<material>Gazebo/Orange</material>
 	</gazebo>
 	<!-- Interial link stores the robot's inertial information -->
-	<link name="$(arg robot_namespace)_inertial_link">
+	<link name="inertial_link">
 		<inertial>
 			<mass value="${chassisMass}" />
@@ -48,20 +48,20 @@
 		</inertial>
 	</link>
-	<joint name="$(arg robot_namespace)_inertial_joint" type="fixed">
+	<joint name="inertial_joint" type="fixed">
 		<origin xyz="0 0 0" rpy="0 0 0" />
-		<parent link="$(arg robot_namespace)_base_link" />
-		<child link="$(arg robot_namespace)_inertial_link" />
+		<parent link="base_link" />
+		<child link="inertial_link" />
 	</joint>
 	<!-- SMB wheel macros -->
-	<xacro:smb_wheel wheel_prefix="$(arg robot_namespace)_LF" BaseNs="$(arg robot_namespace)">
+	<xacro:smb_wheel wheel_prefix="LF">
 		<origin xyz="${frontWheelX} ${chassisWidth/2+wheelClearance+wheelWidth/2} ${-wheelHeight}" rpy="0 0 0" />
 	</xacro:smb_wheel>
-	<xacro:smb_wheel wheel_prefix="$(arg robot_namespace)_RF" BaseNs="$(arg robot_namespace)">
+	<xacro:smb_wheel wheel_prefix="RF">
 		<origin xyz="${frontWheelX} ${-chassisWidth/2-wheelClearance-wheelWidth/2} ${-wheelHeight}" rpy="0 0 0" />
 	</xacro:smb_wheel>
-	<xacro:smb_wheel wheel_prefix="$(arg robot_namespace)_LH" BaseNs="$(arg robot_namespace)">
+	<xacro:smb_wheel wheel_prefix="LH">
 		<origin xyz="${backWheelX} ${chassisWidth/2+wheelClearance+wheelWidth/2} ${-wheelHeight}" rpy="0 0 0" />
 	</xacro:smb_wheel>
-	<xacro:smb_wheel wheel_prefix="$(arg robot_namespace)_RH" BaseNs="$(arg robot_namespace)">
+	<xacro:smb_wheel wheel_prefix="RH">
 		<origin xyz="${backWheelX} ${-chassisWidth/2-wheelClearance-wheelWidth/2} ${-wheelHeight}" rpy="0 0 0" />
 	</xacro:smb_wheel>
@@ -74,5 +74,5 @@
 			<alwaysOn>true</alwaysOn>
 			<updateRate>50.0</updateRate>
-			<bodyName>$(arg robot_namespace)_base_link</bodyName>
+			<bodyName>base_link</bodyName>
 			<topicName>ground_truth/state</topicName>
 			<gaussianNoise>0.001</gaussianNoise>
@@ -83,5 +83,5 @@
 	</gazebo>
 	<xacro:include filename="$(find smb_description)/urdf/sensor_head_2.urdf.xacro"/>
-	<xacro:sensor_head parent="$(arg robot_namespace)_base_link" name="$(arg robot_namespace)_sensor_head">
+	<xacro:sensor_head parent="base_link" name="sensor_head">
 		<origin xyz="0.2 0 0.576" rpy="0 0 0" />
 	</xacro:sensor_head>

File: smb_simulator/smb_description/urdf/wheel.urdf.xacro (robot description, xacro)
@@ -10,5 +10,5 @@
     <xacro:property name="wheelHeight" value="0.05"/>
     <xacro:property name="wheelMass" value="5"/>
-	<xacro:macro name="smb_wheel" params="wheel_prefix *joint_pose">
+	<xacro:macro name="smb_wheel" params="wheel_prefix *joint_pose BaseNs">
 		<link name="${wheel_prefix}_WHEEL_LINK">
 			<inertial>
@@ -43,5 +43,5 @@
 		</gazebo>
 		<joint name="${wheel_prefix}_WHEEL" type="continuous">
-			<parent link="base_link"/>
+			<parent link="${BaseNs}_base_link"/>
 			<child link="${wheel_prefix}_WHEEL_LINK"/>
 			<xacro:insert_block name="joint_pose"/>
