Commit message: ReviseFrameOfVelodyneWhilePublishPoints. 20241105

File: lidar_simulator/lidar_description/urdf/VLP-16-2.urdf.xacro (robot description, xacro)
@@ -2,5 +2,5 @@
 <robot xmlns:xacro="http://www.ros.org/wiki/xacro" name="VLP-16">
   <xacro:property name="M_PI" value="3.1415926535897931" />
-  <xacro:macro name="VLP-16" params="*origin parent:=base_link name:=velodyne topic:=/velodyne_points hz:=10 lasers:=16 samples:=1875 collision_range:=0.8 min_range:=0.9 max_range:=130.0 noise:=0.008 min_angle:=-${M_PI} max_angle:=${M_PI} gpu:=false">
+  <xacro:macro name="VLP-16" params="*origin parent:=base_link name:=velodyne topic:=/velodyne_points hz:=10 lasers:=16 samples:=1875 collision_range:=0.8 min_range:=0.9 max_range:=130.0 noise:=0.008 min_angle:=-${M_PI} max_angle:=${M_PI} gpu:=false RobotNs:=robot">
     <joint name="${name}_base_mount_joint" type="fixed">
       <xacro:insert_block name="origin" />
@@ -51,4 +51,17 @@
       </visual>
     </link>
+    <!-- AddRobotNsAsFrameNs -->
+    <joint name="${name}_base_scan_joint_for_supplementation" type="fixed">
+		  <origin xyz="0 0 0" rpy="0 0 0"/>
+		  <parent link="${name}" />
+		  <child link="${RobotNs}/${name}"/>
+	  </joint>
+    <link name="${RobotNs}/${name}">
+			<inertial>
+				<mass value="0.001" />
+				<origin xyz="0 0 0" rpy="0 0 0"/>
+				<inertia ixx="0" ixy="0" ixz="0" iyy="0" iyz="0" izz="0" />
+			</inertial>
+		</link>
     <!-- Gazebo requires the velodyne_gazebo_plugins package -->
     <gazebo reference="${name}">

File: smb_simulator/smb_description/urdf/sensor_head_2.urdf.xacro (robot description, xacro)
@@ -1,5 +1,5 @@
 <?xml version="1.0"?>
 <robot xmlns:xacro="http://www.ros.org/wiki/xacro" name="sensor_head">
-	<xacro:macro name="sensor_head" params="*origin parent:=base_link name:=sensor_head">
+	<xacro:macro name="sensor_head" params="*origin parent:=base_link name:=sensor_head RobotNs:=robot">
 		<joint name="${name}_base_mount_joint" type="fixed">
 			<xacro:insert_block name="origin" />
@@ -16,5 +16,5 @@
 		<xacro:arg name="gpu" default="true"/>
 		<xacro:include filename="$(find lidar_description)/urdf/VLP-16-2.urdf.xacro"/>
-		<xacro:VLP-16 parent="${name}_base_link" name="${name}_velodyne" topic="${name}_velodyne_points" hz="10" lasers="32" samples="440" gpu="$(arg gpu)" collision_range="0.2" min_range="0.2">
+		<xacro:VLP-16 parent="${name}_base_link" name="${name}_velodyne" topic="${name}_velodyne_points" hz="10" lasers="32" samples="440" gpu="$(arg gpu)" collision_range="0.2" min_range="0.2" RobotNs="${RobotNs}">
 			<origin xyz="0.03 0 0.08" rpy="0 0 0" />
 		</xacro:VLP-16>

File: smb_simulator/smb_description/urdf/smb.urdf.xacro (robot description, xacro)
@@ -83,5 +83,5 @@
 	</gazebo>
 	<xacro:include filename="$(find smb_description)/urdf/sensor_head_2.urdf.xacro"/>
-	<xacro:sensor_head parent="$(arg robot_namespace)_base_link" name="$(arg robot_namespace)_sensor_head">
+	<xacro:sensor_head parent="$(arg robot_namespace)_base_link" name="$(arg robot_namespace)_sensor_head" RobotNs="$(arg robot_namespace)">
 		<origin xyz="0.2 0 0.576" rpy="0 0 0" />
 	</xacro:sensor_head>

Commit message: Add a new environment with closed third floor environment for Smb simulation env 1. Besides, add a new lidar for smb. In addition, adjust the friction param of the StairEnvironment5 in the env 3. 20260109.

File: lidar_simulator/lidar_description/urdf/VLP-16-2.urdf.xacro (robot description, xacro)
@@ -51,5 +51,5 @@
       </visual>
     </link>
-    <!-- AddRobotNsAsFrameNs -->
+    <!-- AddRobotNsAsFrameNs. Written by December. -->
     <joint name="${name}_base_scan_joint_for_supplementation" type="fixed">
 		  <origin xyz="0 0 0" rpy="0 0 0"/>

File: smb_simulator/smb_description/urdf/SensorHead.urdf.xacro (robot description, xacro)
@@ -16,6 +16,9 @@
 		<xacro:arg name="gpu" default="true"/>
 		<xacro:include filename="$(find lidar_description)/urdf/VLP-16-2.urdf.xacro"/>
-		<xacro:VLP-16 parent="${name}_base_link" name="${name}_Top_Velodyne" topic="${name}_Top_Velodyne_Points" hz="10" lasers="32" samples="20000" gpu="$(arg gpu)" collision_range="0.2" min_range="0.2" RobotNs="${RobotNs}">
+		<xacro:VLP-16 parent="${name}_base_link" name="${name}_Top_Velodyne" topic="${name}_Top_Velodyne_Points" hz="5" lasers="32" samples="2000" gpu="$(arg gpu)" collision_range="0.2" min_range="0.2" RobotNs="${RobotNs}">
 			<origin xyz="0.03 0 0.08" rpy="0 0 0" />
+		</xacro:VLP-16>
+		<xacro:VLP-16 parent="${name}_base_link" name="${name}_Side_Velodyne" topic="${name}_Side_Velodyne_Points" hz="5" lasers="32" samples="2000" gpu="$(arg gpu)" collision_range="0.2" min_range="0.9" RobotNs="${RobotNs}">
+			<origin xyz="-0.1 0.2 -0.05" rpy="-1.57 0 0" />
 		</xacro:VLP-16>
 		<!-- <xacro:VLP-16 parent="${name}_base_link" name="${name}_Front_Velodyne" topic="${name}_Front_Velodyne_Points" hz="10" lasers="32" samples="440" gpu="false" collision_range="0.2" min_range="0.7" RobotNs="${RobotNs}">
