Commit message: Revise UnitreeA1 Sensor Head Model. 20241106.

File: lidar_simulator/lidar_description/urdf/VLP-16-ForUnitreeA1.urdf.xacro (robot description, xacro)
@@ -10,9 +10,9 @@
     <link name="${name}_base_link">
       <inertial>
-        <mass value="0.83"/>
+        <mass value="0.0000083"/>
         <origin xyz="0 0 0.03585"/>
-        <inertia ixx="${(0.83 * (3.0*0.0516*0.0516 + 0.0717*0.0717)) / 12.0}" ixy="0" ixz="0"
-          iyy="${(0.83 * (3.0*0.0516*0.0516 + 0.0717*0.0717)) / 12.0}" iyz="0"
-          izz="${0.5 * 0.83 * (0.0516*0.0516)}"/>
+        <inertia ixx="${(0.0000083 * (3.0*0.0516*0.0516 + 0.0717*0.0717)) / 12.0}" ixy="0" ixz="0"
+          iyy="${(0.0000083 * (3.0*0.0516*0.0516 + 0.0717*0.0717)) / 12.0}" iyz="0"
+          izz="${0.5 * 0.0000083 * (0.0516*0.0516)}"/>
       </inertial>
       <visual>
@@ -40,7 +40,7 @@
     <link name="${name}">
       <inertial>
-        <mass value="0.01"/>
+        <mass value="0.0000001"/>
         <origin xyz="0 0 0"/>
-        <inertia ixx="1e-7" ixy="0" ixz="0" iyy="1e-7" iyz="0" izz="1e-7"/>
+        <inertia ixx="1e-12" ixy="0" ixz="0" iyy="1e-12" iyz="0" izz="1e-12"/>
       </inertial>
       <visual>

File: unitree_simulator/unitree_ros/robots/a1_description/xacro/SensorHeadForUnitreeA1.urdf.xacro (robot description, xacro)
@@ -16,6 +16,6 @@
 		<xacro:arg name="gpu" default="true"/>
 		<xacro:include filename="$(find lidar_description)/urdf/VLP-16-ForUnitreeA1.urdf.xacro"/>
-		<xacro:VLP-16 parent="${name}_base_link" name="${name}_Top_Velodyne" topic="${name}_Top_Velodyne_Points" hz="10" lasers="32" samples="440" gpu="$(arg gpu)" collision_range="0.2" min_range="0.39">
-			<origin xyz="0.00 0 0.03" rpy="0 0 0" />
+		<xacro:VLP-16 parent="${name}_base_link" name="${name}_Top_Velodyne" topic="${name}_Top_Velodyne_Points" hz="10" lasers="32" samples="440" gpu="$(arg gpu)" collision_range="0.2" min_range="0.2">
+			<origin xyz="0.10 0 0.12" rpy="0 0 0" />
 		</xacro:VLP-16>
 		<!-- <xacro:VLP-16 parent="${name}_base_link" name="${name}_Front_Velodyne" topic="${name}_Front_Velodyne_Points" hz="10" lasers="32" samples="440" gpu="false" collision_range="0.2" min_range="0.7">

Commit message: Adjust the lidar simulator by adding an config of 'organizePoinycloud'. Besids, adjust the world param - changing the frequency from 1000 to 10000. Finally, adjust the param of the gazebo mpc controller for the unitree A1- the gait counter for calculating the phase of the swing leg. 20260114.

File: lidar_simulator/lidar_description/urdf/VLP-16-ForUnitreeA1.urdf.xacro (robot description, xacro)
@@ -2,5 +2,5 @@
 <robot xmlns:xacro="http://www.ros.org/wiki/xacro" name="VLP-16">
   <xacro:property name="M_PI" value="3.1415926535897931" />
-  <xacro:macro name="VLP-16" params="*origin parent:=base_link name:=velodyne topic:=/velodyne_points hz:=10 lasers:=16 samples:=1875 collision_range:=0.8 min_range:=0.9 max_range:=130.0 noise:=0.008 min_angle:=-${M_PI} max_angle:=${M_PI} gpu:=false">
+  <xacro:macro name="VLP-16" params="*origin parent:=base_link name:=velodyne topic:=/velodyne_points hz:=10 lasers:=16 samples:=1875 collision_range:=0.8 min_range:=0.9 max_range:=130.0 noise:=0.008 min_angle:=-${M_PI} max_angle:=${M_PI} gpu:=false organize_pointcloud:=false">
     <joint name="${name}_base_mount_joint" type="fixed">
       <xacro:insert_block name="origin" />
@@ -90,4 +90,5 @@
             <max_range>${max_range}</max_range>
             <gaussianNoise>${noise}</gaussianNoise>
+            <organizePointcloud>${organize_pointcloud}</organizePointcloud>
           </plugin>
         </sensor>
@@ -130,4 +131,5 @@
             <max_range>${max_range}</max_range>
             <gaussianNoise>${noise}</gaussianNoise>
+            <organizePointcloud>${organize_pointcloud}</organizePointcloud>
           </plugin>
         </sensor>

File: unitree_simulator/unitree_ros/robots/a1_description/xacro/SensorHeadForUnitreeA1.urdf.xacro (robot description, xacro)
@@ -16,6 +16,9 @@
 		<xacro:arg name="gpu" default="true"/>
 		<xacro:include filename="$(find lidar_description)/urdf/VLP-16-ForUnitreeA1.urdf.xacro"/>
-		<xacro:VLP-16 parent="${name}_base_link" name="${name}_Top_Velodyne" topic="${name}_Top_Velodyne_Points" hz="10" lasers="32" samples="440" gpu="$(arg gpu)" collision_range="0.2" min_range="0.2">
-			<origin xyz="0.10 0 0.12" rpy="0 0 0" />
+		<xacro:VLP-16 parent="${name}_base_link" name="${name}_Top_Velodyne" topic="${name}_Top_Velodyne_Points" hz="5" lasers="32" samples="440" gpu="$(arg gpu)" collision_range="0.2" min_range="0.5" max_range="20.0" organize_pointcloud="true">
+			<origin xyz="0.10 0 0.07" rpy="0 0 0" />
+		</xacro:VLP-16>
+		<xacro:VLP-16 parent="${name}_base_link" name="${name}_Side_Velodyne" topic="${name}_Side_Velodyne_Points" hz="5" lasers="32" samples="440" gpu="$(arg gpu)" collision_range="0.2" min_range="0.6" max_range="20.0" organize_pointcloud="true">
+			<origin xyz="0.10 -0.05 0.20" rpy="-1.57 0 0" />
 		</xacro:VLP-16>
 		<!-- <xacro:VLP-16 parent="${name}_base_link" name="${name}_Front_Velodyne" topic="${name}_Front_Velodyne_Points" hz="10" lasers="32" samples="440" gpu="false" collision_range="0.2" min_range="0.7">
