Commit message: Add a fix stand controller into the a1\_cpp project (The controller for the unitree A1.) and this adjustment would make the robot could walk in the ode frequency 1000. Besides, adjust the mass (parameter) of the realsense d435 camera. Finally, the cmakelists file of the unitree\_guide has been adjusted to make the junior controller are compiled for the unitree A1. 20260110.

File: realsense_simulator/xacro/depthcam.xacro (robot description, xacro)
@@ -10,5 +10,5 @@
     <xacro:property name="d435_cam_height" value="0.025"/>
     <xacro:property name="d435_cam_depth" value="0.02505"/>
-    <xacro:property name="d435_cam_mass" value="0.564"/>
+    <xacro:property name="d435_cam_mass" value="0.000000564"/>
     <xacro:property name="d435_cam_mount_from_center_offset" value="0.0149"/>
     <xacro:property name="d435_cam_depth_px" value="${d435_cam_mount_from_center_offset}"/>
